Commit message: non-kdl-solver

File: src/lab_2/xacro/3_degree_robot.xacro (robot description, xacro)
@@ -21,9 +21,18 @@
     <xacro:property name="z2" value="${yaml_params['z2']}" />
     <xacro:property name="z3" value="${yaml_params['z3']}" />
+    <material name="red">
+      <color rgba="0.80392157 0 0 1"/>
+    </material>
+    <material name="blue">
+      <color rgba="0 0.1 0.7 1"/>
+    </material>
+    <material name="black">
+      <color rgba="0.05 0.05 0.05 1"/>
+    </material>
     <xacro:macro name="link_" params="name">
         <link name="${name}">
            <visual>
             <geometry>
-              <cylinder radius="0.2" length="0.5"/>
+              <cylinder radius="0.05" length="0.1"/>
             </geometry>
             <origin xyz="0 0 0" rpy="0 0 1"/>
