Commit message: zmiana na python2.7, zeby uzyt ros.tf.transforms

File: src/lab_2/urdf/urdf_from_xacro.urdf (robot description, URDF)
Before this commit: robot robot_from_DH_table, 5 links, 4 joints
Joints:
- joint base_link_to_link_0: type continuous -> fixed
- joint link_1_to_link_2: origin xyz=0.0 -0.0 0.0 rpy=-1.57 -0.0 0.0 -> xyz=0.0 0.0 0.0 rpy=-1.57 -0.0 0.0
- joint link_2_to_link_3: origin xyz=2.0 0.0 0.0 rpy=0.0 -0.0 0.0 -> xyz=1.0 0.0 0.0 rpy=0.0 -0.0 0.0

File: src/lab_2/xacro/test.xacro (robot description, xacro)
@@ -27,11 +27,11 @@
               <cylinder radius="0.2" length="0.5"/>
             </geometry>
-            <origin xyz="0 0 1" rpy="0 0 0"/>
+            <origin xyz="0 0 0" rpy="0 0 1"/>
             <material name="blue"/>
           </visual>
         </link>
     </xacro:macro>
-    <xacro:macro name="joint_" params="parent child x y z roll pitch yaw">
-        <joint name="${parent}_to_${child}" type="continuous">
+    <xacro:macro name="joint_" params="parent child x y z roll pitch yaw type">
+        <joint name="${parent}_to_${child}" type="${type}">
             <parent link="${parent}"/>
             <child link="${child}"/>
@@ -43,9 +43,9 @@
     <xacro:link_ name="link_0" />
     <xacro:link_ name="link_1" />
-    <xacro:joint_ parent="base_link" child="link_0" x="0" y="0" z="0" roll="0" pitch="0" yaw="0" />
-    <xacro:joint_ parent="link_0" child="link_1" x="${x1}" y="${y1}" z="${z1}" roll="${roll1}" pitch="${pitch1}" yaw="${yaw1}" />
+    <xacro:joint_ parent="base_link" child="link_0" x="0" y="0" z="0" roll="0" pitch="0" yaw="0" type="fixed" />
+    <xacro:joint_ parent="link_0" child="link_1" x="${x1}" y="${y1}" z="${z1}" roll="${roll1}" pitch="${pitch1}" yaw="${yaw1}" type="continuous" />
     <xacro:link_ name="link_2" />
-    <xacro:joint_ parent="link_1" child="link_2" x="${x2}" y="${y2}" z="${z2}" roll="${roll2}" pitch="${pitch2}" yaw="${yaw2}" />
+    <xacro:joint_ parent="link_1" child="link_2" x="${x2}" y="${y2}" z="${z2}" roll="${roll2}" pitch="${pitch2}" yaw="${yaw2}" type="continuous"/>
     <xacro:link_ name="link_3" />
-    <xacro:joint_ parent="link_2" child="link_3" x="${x3}" y="${y3}" z="${z3}" roll="${roll3}" pitch="${pitch3}" yaw="${yaw3}" />
+    <xacro:joint_ parent="link_2" child="link_3" x="${x3}" y="${y3}" z="${z3}" roll="${roll3}" pitch="${pitch3}" yaw="${yaw3}" type="continuous"/>
 </robot>
